Commit message: Updated gazebo and URDF file

File: Control/turtle/gazebo/turtle.gazebo.xacro (robot description, xacro)
@@ -7,16 +7,17 @@
       </plugin>
       <plugin filename="gz_ros2_control-system" name="gz_ros2_control::GazeboSimROS2ControlPlugin">
-        <parameters>$(find turtle)/config/joint_controllers.yaml</parameters>
+        <parameters>$(find turtle_on_land_demo)/config/joint_controllers.yaml</parameters>
       </plugin>
     </gazebo>
     <gazebo reference="Sensor_link">
       <sensor name="gpu_lidar" type="gpu_lidar">
+       <pose>0 0 0.5 0 0 0</pose>
           <gz_frame_id>Sensor_link</gz_frame_id>
           <topic>scan</topic>
-          <update_rate>10</update_rate>
+          <update_rate>5</update_rate>
           <lidar>
             <scan>
               <horizontal>
-                <samples>2800</samples>
+                <samples>270</samples>
                 <resolution>1</resolution>
                 <min_angle>-3.14</min_angle>
@@ -24,13 +25,48 @@
               </horizontal>
               <vertical>
-                <samples>1</samples>
-                <resolution>0.1</resolution>
-                <min_angle>0.0</min_angle>
-                <max_angle>0.0</max_angle>
+                <samples>45</samples>
+                <resolution>1</resolution>
+                <min_angle>-0.349066</min_angle>
+                <max_angle>0.785</max_angle>
               </vertical>
             </scan>
             <range>
               <min>0.2</min>
-              <max>3.0</max>
+              <max>30.0</max>
+              <resolution>0.01</resolution>
+            </range>
+            <frame_id>Sensor_link</frame_id>
+          </lidar>
+          <alwaysOn>true</alwaysOn>
+          <visualize>true</visualize>
+        <sensor name="imu_sensor" type="imu">
+          <always_on>1</always_on>
+          <update_rate>1</update_rate>
+          <visualize>true</visualize>
+        <topic>imu</topic>
+      </sensor>
+      </sensor>
+      <sensor name="gpu2_lidar" type="gpu_lidar">
+          <gz_frame_id>Sensor_link</gz_frame_id>
+          <topic>scan2</topic>
+          <update_rate>5</update_rate>
+          <lidar>
+            <scan>
+              <horizontal>
+                <samples>500</samples>
+                <resolution>1</resolution>
+                <min_angle>-0.</min_angle>
+                <max_angle>0.785</max_angle>
+              </horizontal>
+              <vertical>
+                <samples>1</samples>
+                <resolution>1</resolution>
+                <min_angle>-0</min_angle>
+                <max_angle>0</max_angle>
+              </vertical>
+            </scan>
+            <range>
+              <min>0.2</min>
+              <max>30.0</max>
               <resolution>0.01</resolution>
             </range>

File: Control/turtle/urdf/URDF1.urdf.xacro (robot description, xacro)
@@ -2,8 +2,8 @@
 <!-- Turtle on land URDF file-->
 <robot name="URDF1" xmlns:xacro="http://www.ros.org/wiki/xacro">
-  <!-- Import turtle ros2_control description -->
-  <xacro:include filename="$(find turtle)/src/ros2_control.xacro" />
+  <!-- Import turtlebot ros2_control description -->
+  <xacro:include filename="$(find turtle_on_land_demo)/src/ros2_control.xacro" />
   <!-- Import turtle gazebo lidar description -->
-  <xacro:include filename="$(find turtle)/gazebo/turtle.gazebo.xacro" />
+  <xacro:include filename="$(find turtle_on_land_demo)/gazebo/turtle.gazebo.xacro" />
   <!--Link1; Turtle Shell bottom-->
   <link name="base_footprint">
@@ -41,5 +41,5 @@
         <!--Mass parameter for link-->
       <mass
-        value="0.37301" />
+        value="10.97301" />
         <!--Inertial properties-->
       <inertia
@@ -58,5 +58,5 @@
         <!--Filepath to STL visual Mesh file-->
       <geometry>
-        <mesh filename="package://turtle/meshes/visual/base_link.STL"/>
+        <mesh filename="package://turtle_on_land_demo/meshes/visual/base_link.STL"/>
       </geometry>
       <material
@@ -75,5 +75,5 @@
       <geometry>
         <mesh
-          filename="package://turtle/meshes/visual/base_link.STL" />
+          filename="package://turtle_on_land_demo/meshes/visual/base_link.STL" />
       </geometry>
     </collision>
@@ -104,19 +104,19 @@
       <geometry>
         <mesh
-          filename="package://turtle/meshes/visual/Front_right1.STL" />
-      </geometry>
-      <material
-        name="">
-        <color
-          rgba="0 1 0 1" />
-      </material>
-    </visual>
-    <collision>
-      <origin
-        xyz="0 0 0"
-        rpy="0 0 0" />
-      <geometry>
-        <mesh
-          filename="package://turtle/meshes/visual/Front_right1.STL" />
+          filename="package://turtle_on_land_demo/meshes/visual/Front_right1.STL" />
+      </geometry>
+      <material
+        name="">
+        <color
+          rgba="0 1 0 1" />
+      </material>
+    </visual>
+    <collision>
+      <origin
+        xyz="0 0 0"
+        rpy="0 0 0" />
+      <geometry>
+        <mesh
+          filename="package://turtle_on_land_demo/meshes/visual/Front_right1.STL" />
       </geometry>
     </collision>
@@ -138,6 +138,6 @@
       lower="-0.7854"
       upper="0.7854"
-      effort="2"
-      velocity="5" />
+      effort="20"
+      velocity="999" />
     <dynamics damping="0.1" friction="0.1"/>
   </joint>
@@ -165,19 +165,19 @@
       <geometry>
         <mesh
-          filename="package://turtle/meshes/visual/Front_right2.STL" />
-      </geometry>
-      <material
-        name="">
-        <color
-          rgba="0 1 0 1" />
-      </material>
-    </visual>
-    <collision>
-      <origin
-        xyz="0 0 0"
-        rpy="0 0 0" />
-      <geometry>
-        <mesh
-          filename="package://turtle/meshes/visual/Front_right2.STL" />
+          filename="package://turtle_on_land_demo/meshes/visual/Front_right2.STL" />
+      </geometry>
+      <material
+        name="">
+        <color
+          rgba="0 1 0 1" />
+      </material>
+    </visual>
+    <collision>
+      <origin
+        xyz="0 0 0"
+        rpy="0 0 0" />
+      <geometry>
+        <mesh
+          filename="package://turtle_on_land_demo/meshes/visual/Front_right2.STL" />
       </geometry>
     </collision>
@@ -197,8 +197,8 @@
       xyz="0 0 1" />
     <limit
-      lower="-0.2618"
-      upper="0.2618"
-      effort="2"
-      velocity="5" />
+      lower="-0.785398"
+      upper="0.223599"
+      effort="20"
+      velocity="999" />
     <dynamics damping="0.1" friction="0.1"/>
   </joint>
@@ -226,19 +226,19 @@
       <geometry>
         <mesh
-          filename="package://turtle/meshes/visual/Back_right1.STL" />
-      </geometry>
-      <material
-        name="">
-        <color
-          rgba="0 1 0 1" />
-      </material>
-    </visual>
-    <collision>
-      <origin
-        xyz="0 0 0"
-        rpy="0 0 0" />
-      <geometry>
-        <mesh
-          filename="package://turtle/meshes/visual/Back_right1.STL" />
+          filename="package://turtle_on_land_demo/meshes/visual/Back_right1.STL" />
+      </geometry>
+      <material
+        name="">
+        <color
+          rgba="0 1 0 1" />
+      </material>
+    </visual>
+    <collision>
+      <origin
+        xyz="0 0 0"
+        rpy="0 0 0" />
+      <geometry>
+        <mesh
+          filename="package://turtle_on_land_demo/meshes/visual/Back_right1.STL" />
       </geometry>
     </collision>
@@ -260,6 +260,6 @@
       lower="-0.7854"
       upper="0.7854"
-      effort="2"
-      velocity="5" />
+      effort="10"
+      velocity="999" />
     <dynamics damping="0.1" friction="0.1"/>
   </joint>
@@ -287,19 +287,19 @@
       <geometry>
         <mesh
-          filename="package://turtle/meshes/visual/Back_right2.STL" />
-      </geometry>
-      <material
-        name="">
-        <color
-          rgba="0 1 0 1" />
-      </material>
-    </visual>
-    <collision>
-      <origin
-        xyz="0 0 0"
-        rpy="0 0 0" />
-      <geometry>
-        <mesh
-          filename="package://turtle/meshes/visual/Back_right2.STL" />
+          filename="package://turtle_on_land_demo/meshes/visual/Back_right2.STL" />
+      </geometry>
+      <material
+        name="">
+        <color
+          rgba="0 1 0 1" />
+      </material>
+    </visual>
+    <collision>
+      <origin
+        xyz="0 0 0"
+        rpy="0 0 0" />
+      <geometry>
+        <mesh
+          filename="package://turtle_on_land_demo/meshes/visual/Back_right2.STL" />
       </geometry>
     </collision>
@@ -319,8 +319,8 @@
       xyz="0 0 1" />
     <limit
-      lower="-0.2618"
-      upper="0.2618"
-      effort="2"
-      velocity="5" />
+      lower="-0.785398"
+      upper="0.223599"
+      effort="10"
+      velocity="999" />
     <dynamics damping="0.1" friction="0.1"/>
   </joint>
@@ -348,19 +348,19 @@
       <geometry>
         <mesh
-          filename="package://turtle/meshes/visual/Front_left1.STL" />
-      </geometry>
-      <material
-        name="">
-        <color
-          rgba="0 1 0 1" />
-      </material>
-    </visual>
-    <collision>
-      <origin
-        xyz="0 0 0"
-        rpy="0 0 0" />
-      <geometry>
-        <mesh
-          filename="package://turtle/meshes/visual/Front_left1.STL" />
+          filename="package://turtle_on_land_demo/meshes/visual/Front_left1.STL" />
+      </geometry>
+      <material
+        name="">
+        <color
+          rgba="0 1 0 1" />
+      </material>
+    </visual>
+    <collision>
+      <origin
+        xyz="0 0 0"
+        rpy="0 0 0" />
+      <geometry>
+        <mesh
+          filename="package://turtle_on_land_demo/meshes/visual/Front_left1.STL" />
       </geometry>
     </collision>
@@ -382,6 +382,6 @@
       lower="-0.6854"
       upper="0.6854"
-      effort="2"
-      velocity="5" />
+      effort="20"
+      velocity="999" />
     <dynamics damping="0.1" friction="0.1"/>
   </joint>
@@ -409,19 +409,19 @@
       <geometry>
         <mesh
-          filename="package://turtle/meshes/visual/Front_left2.STL" />
-      </geometry>
-      <material
-        name="">
-        <color
-          rgba="0 1 0 1" />
-      </material>
-    </visual>
-    <collision>
-      <origin
-        xyz="0 0 0"
-        rpy="0 0 0" />
-      <geometry>
-        <mesh
-          filename="package://turtle/meshes/visual/Front_left2.STL" />
+          filename="package://turtle_on_land_demo/meshes/visual/Front_left2.STL" />
+      </geometry>
+      <material
+        name="">
+        <color
+          rgba="0 1 0 1" />
+      </material>
+    </visual>
+    <collision>
+      <origin
+        xyz="0 0 0"
+        rpy="0 0 0" />
+      <geometry>
+        <mesh
+          filename="package://turtle_on_land_demo/meshes/visual/Front_left2.STL" />
       </geometry>
     </collision>
@@ -441,8 +441,8 @@
       xyz="0 0 1" />
     <limit
-      lower="-0.2618"
-      upper="0.2618"
-      effort="2"
-      velocity="5" />
+      lower="-0.223599"
+      upper="0.785398"
+      effort="20"
+      velocity="999" />
     <dynamics damping="0.1" friction="0.1"/>
   </joint>
@@ -470,19 +470,19 @@
       <geometry>
         <mesh
-          filename="package://turtle/meshes/visual/Back_left1.STL" />
-      </geometry>
-      <material
-        name="">
-        <color
-          rgba="0 1 0 1" />
-      </material>
-    </visual>
-    <collision>
-      <origin
-        xyz="0 0 0"
-        rpy="0 0 0" />
-      <geometry>
-        <mesh
-          filename="package://turtle/meshes/visual/Back_left1.STL" />
+          filename="package://turtle_on_land_demo/meshes/visual/Back_left1.STL" />
+      </geometry>
+      <material
+        name="">
+        <color
+          rgba="0 1 0 1" />
+      </material>
+    </visual>
+    <collision>
+      <origin
+        xyz="0 0 0"
+        rpy="0 0 0" />
+      <geometry>
+        <mesh
+          filename="package://turtle_on_land_demo/meshes/visual/Back_left1.STL" />
       </geometry>
     </collision>
@@ -504,6 +504,6 @@
       lower="-0.7854"
       upper="0.7854"
-      effort="2"
-      velocity="5" />
+      effort="10"
+      velocity="999" />
     <dynamics damping="0.1" friction="0.1"/>
   </joint>
@@ -531,19 +531,19 @@
       <geometry>
         <mesh
-          filename="package://turtle/meshes/visual/Back_left2.STL" />
-      </geometry>
-      <material
-        name="">
-        <color
-          rgba="0 1 0 1" />
-      </material>
-    </visual>
-    <collision>
-      <origin
-        xyz="0 0 0"
-        rpy="0 0 0" />
-      <geometry>
-        <mesh
-          filename="package://turtle/meshes/visual/Back_left2.STL" />
+          filename="package://turtle_on_land_demo/meshes/visual/Back_left2.STL" />
+      </geometry>
+      <material
+        name="">
+        <color
+          rgba="0 1 0 1" />
+      </material>
+    </visual>
+    <collision>
+      <origin
+        xyz="0 0 0"
+        rpy="0 0 0" />
+      <geometry>
+        <mesh
+          filename="package://turtle_on_land_demo/meshes/visual/Back_left2.STL" />
       </geometry>
     </collision>
@@ -563,11 +563,10 @@
       xyz="0 0 1" />
     <limit
-      lower="-0.2618"
-      upper="0.2618"
-      effort="2"
-      velocity="5" />
-    <dynamics damping="0.1" friction="0.1"/>
-  </joint>
-<!--Sesnor_Link-->
+      lower="-0.223599"
+      upper="0.785398"
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