Commit message: Updated publisher file, subscribes to topic "cmd_vel", URDF friction , 0.1 -> 5 , ros2_control without redundant code

File: Control/turtle/src/ros2_control.xacro (robot description, xacro)
@@ -102,12 +102,3 @@
       </joint>
     </ros2_control>
-  <!-- =============== Gazebo =============== -->
-    <gazebo>
-      <plugin filename="gz_ros2_control-system" name="gz_ros2_control::GazeboSimROS2ControlPlugin">
-        <parameters>$(find turtle)/config/joint_controllers.yaml</parameters>
-      </plugin>
-    </gazebo>
-    <plugin name="lidar" filename="libgazebo_ros_ray_sensor.so">
-      <output_type> sensor_msgs/LaserScan</output_type>
-    </plugin>
 </robot>

File: Control/turtle/urdf/URDF1.urdf.xacro (robot description, xacro)
@@ -3,7 +3,7 @@
 <robot name="URDF1" xmlns:xacro="http://www.ros.org/wiki/xacro">
   <!-- Import turtle ros2_control description -->
-  <xacro:include filename="$(find turtle)/src/ros2_control.xacro" />
-  <!-- Import turtle gazebo lidar description -->
-  <xacro:include filename="$(find turtle)/gazebo/turtle.gazebo.xacro" />
+  <xacro:include filename="$(find turtle_on_land_demo)/src/ros2_control.xacro" />
+  <!-- Import turtle gazebo sensor descriptions -->
+  <xacro:include filename="$(find turtle_on_land_demo)/gazebo/turtle.gazebo.xacro" />
   <!--Link1; Turtle Shell bottom-->
   <link name="base_footprint">
@@ -28,5 +28,5 @@
       <!--Child link defining child frame-->
       <child link="base_link" />
-      <dynamics damping="0.1" friction="0.01"/>
+      <dynamics damping="0.1" friction="5"/>
   </joint>
   <!--Joint parameters are the same throughout for each link connection-->
@@ -41,5 +41,5 @@
         <!--Mass parameter for link-->
       <mass
-        value="0.37301" />
+        value="10.97301" />
         <!--Inertial properties-->
       <inertia
@@ -58,5 +58,5 @@
         <!--Filepath to STL visual Mesh file-->
       <geometry>
-        <mesh filename="package://turtle/meshes/visual/base_link.STL"/>
+        <mesh filename="package://turtle_on_land_demo/meshes/visual/base_link.STL"/>
       </geometry>
       <material
@@ -75,5 +75,5 @@
       <geometry>
         <mesh
-          filename="package://turtle/meshes/visual/base_link.STL" />
+          filename="package://turtle_on_land_demo/meshes/visual/base_link.STL" />
       </geometry>
     </collision>
@@ -104,19 +104,19 @@
       <geometry>
         <mesh
-          filename="package://turtle/meshes/visual/Front_right1.STL" />
-      </geometry>
-      <material
-        name="">
-        <color
-          rgba="0 1 0 1" />
-      </material>
-    </visual>
-    <collision>
-      <origin
-        xyz="0 0 0"
-        rpy="0 0 0" />
-      <geometry>
-        <mesh
-          filename="package://turtle/meshes/visual/Front_right1.STL" />
+          filename="package://turtle_on_land_demo/meshes/visual/Front_right1.STL" />
+      </geometry>
+      <material
+        name="">
+        <color
+          rgba="0 1 0 1" />
+      </material>
+    </visual>
+    <collision>
+      <origin
+        xyz="0 0 0"
+        rpy="0 0 0" />
+      <geometry>
+        <mesh
+          filename="package://turtle_on_land_demo/meshes/visual/Front_right1.STL" />
       </geometry>
     </collision>
@@ -138,7 +138,7 @@
       lower="-0.7854"
       upper="0.7854"
-      effort="2"
-      velocity="5" />
-    <dynamics damping="0.1" friction="0.1"/>
+      effort="20"
+      velocity="999" />
+    <dynamics damping="0.1" friction="5"/>
   </joint>
   <!--Link4; Froint right flipper-->
@@ -165,19 +165,19 @@
       <geometry>
         <mesh
-          filename="package://turtle/meshes/visual/Front_right2.STL" />
-      </geometry>
-      <material
-        name="">
-        <color
-          rgba="0 1 0 1" />
-      </material>
-    </visual>
-    <collision>
-      <origin
-        xyz="0 0 0"
-        rpy="0 0 0" />
-      <geometry>
-        <mesh
-          filename="package://turtle/meshes/visual/Front_right2.STL" />
+          filename="package://turtle_on_land_demo/meshes/visual/Front_right2.STL" />
+      </geometry>
+      <material
+        name="">
+        <color
+          rgba="0 1 0 1" />
+      </material>
+    </visual>
+    <collision>
+      <origin
+        xyz="0 0 0"
+        rpy="0 0 0" />
+      <geometry>
+        <mesh
+          filename="package://turtle_on_land_demo/meshes/visual/Front_right2.STL" />
       </geometry>
     </collision>
@@ -197,9 +197,9 @@
       xyz="0 0 1" />
     <limit
-      lower="-0.2618"
-      upper="0.2618"
-      effort="2"
-      velocity="5" />
-    <dynamics damping="0.1" friction="0.1"/>
+      lower="-0.785398"
+      upper="0.223599"
+      effort="20"
+      velocity="999" />
+    <dynamics damping="0.1" friction="5"/>
   </joint>
   <!--Link5; Back right shoulder-->
@@ -226,19 +226,19 @@
       <geometry>
         <mesh
-          filename="package://turtle/meshes/visual/Back_right1.STL" />
-      </geometry>
-      <material
-        name="">
-        <color
-          rgba="0 1 0 1" />
-      </material>
-    </visual>
-    <collision>
-      <origin
-        xyz="0 0 0"
-        rpy="0 0 0" />
-      <geometry>
-        <mesh
-          filename="package://turtle/meshes/visual/Back_right1.STL" />
+          filename="package://turtle_on_land_demo/meshes/visual/Back_right1.STL" />
+      </geometry>
+      <material
+        name="">
+        <color
+          rgba="0 1 0 1" />
+      </material>
+    </visual>
+    <collision>
+      <origin
+        xyz="0 0 0"
+        rpy="0 0 0" />
+      <geometry>
+        <mesh
+          filename="package://turtle_on_land_demo/meshes/visual/Back_right1.STL" />
       </geometry>
     </collision>
@@ -260,7 +260,7 @@
       lower="-0.7854"
       upper="0.7854"
-      effort="2"
-      velocity="5" />
-    <dynamics damping="0.1" friction="0.1"/>
+      effort="10"
+      velocity="999" />
+    <dynamics damping="0.1" friction="5"/>
   </joint>
   <!--Link6; Back right flipper-->
@@ -287,19 +287,19 @@
       <geometry>
         <mesh
-          filename="package://turtle/meshes/visual/Back_right2.STL" />
-      </geometry>
-      <material
-        name="">
-        <color
-          rgba="0 1 0 1" />
-      </material>
-    </visual>
-    <collision>
-      <origin
-        xyz="0 0 0"
-        rpy="0 0 0" />
-      <geometry>
-        <mesh
-          filename="package://turtle/meshes/visual/Back_right2.STL" />
+          filename="package://turtle_on_land_demo/meshes/visual/Back_right2.STL" />
+      </geometry>
+      <material
+        name="">
+        <color
+          rgba="0 1 0 1" />
+      </material>
+    </visual>
+    <collision>
+      <origin
+        xyz="0 0 0"
+        rpy="0 0 0" />
+      <geometry>
+        <mesh
+          filename="package://turtle_on_land_demo/meshes/visual/Back_right2.STL" />
       </geometry>
     </collision>
@@ -319,9 +319,9 @@
       xyz="0 0 1" />
     <limit
-      lower="-0.2618"
-      upper="0.2618"
-      effort="2"
-      velocity="5" />
-    <dynamics damping="0.1" friction="0.1"/>
+      lower="-0.785398"
+      upper="0.223599"
+      effort="10"
+      velocity="999" />
+    <dynamics damping="0.1" friction="5"/>
   </joint>
   <!--Link7; Front left shoulder-->
@@ -348,19 +348,19 @@
       <geometry>
         <mesh
-          filename="package://turtle/meshes/visual/Front_left1.STL" />
-      </geometry>
-      <material
-        name="">
-        <color
-          rgba="0 1 0 1" />
-      </material>
-    </visual>
-    <collision>
-      <origin
-        xyz="0 0 0"
-        rpy="0 0 0" />
-      <geometry>
-        <mesh
-          filename="package://turtle/meshes/visual/Front_left1.STL" />
+          filename="package://turtle_on_land_demo/meshes/visual/Front_left1.STL" />
+      </geometry>
+      <material
+        name="">
+        <color
+          rgba="0 1 0 1" />
+      </material>
+    </visual>
+    <collision>
+      <origin
+        xyz="0 0 0"
+        rpy="0 0 0" />
+      <geometry>
+        <mesh
+          filename="package://turtle_on_land_demo/meshes/visual/Front_left1.STL" />
       </geometry>
     </collision>
@@ -382,7 +382,7 @@
       lower="-0.6854"
       upper="0.6854"
-      effort="2"
-      velocity="5" />
-    <dynamics damping="0.1" friction="0.1"/>
+      effort="20"
+      velocity="999" />
+    <dynamics damping="0.1" friction="5"/>
   </joint>
   <!--Link8; Front left flipper-->
@@ -409,19 +409,19 @@
       <geometry>
         <mesh
-          filename="package://turtle/meshes/visual/Front_left2.STL" />
-      </geometry>
-      <material
-        name="">
-        <color
-          rgba="0 1 0 1" />
-      </material>
-    </visual>
-    <collision>
-      <origin
-        xyz="0 0 0"
-        rpy="0 0 0" />
-      <geometry>
-        <mesh
-          filename="package://turtle/meshes/visual/Front_left2.STL" />
+          filename="package://turtle_on_land_demo/meshes/visual/Front_left2.STL" />
+      </geometry>
+      <material
+        name="">
+        <color
+          rgba="0 1 0 1" />
+      </material>
+    </visual>
+    <collision>
+      <origin
+        xyz="0 0 0"
+        rpy="0 0 0" />
+      <geometry>
+        <mesh
+          filename="package://turtle_on_land_demo/meshes/visual/Front_left2.STL" />
       </geometry>
     </collision>
@@ -441,9 +441,9 @@
       xyz="0 0 1" />
     <limit
-      lower="-0.2618"
-      upper="0.2618"
-      effort="2"
-      velocity="5" />
-    <dynamics damping="0.1" friction="0.1"/>
+      lower="-0.223599"
+      upper="0.785398"
+      effort="20"
+      velocity="999" />
+    <dynamics damping="0.1" friction="5"/>
   </joint>
   <!--Link9; Back left shoulder-->
@@ -470,19 +470,19 @@
       <geometry>
         <mesh
-          filename="package://turtle/meshes/visual/Back_left1.STL" />
-      </geometry>
-      <material
-        name="">
-        <color
-          rgba="0 1 0 1" />
-      </material>
-    </visual>
-    <collision>
-      <origin
-        xyz="0 0 0"
-        rpy="0 0 0" />
-      <geometry>
-        <mesh
-          filename="package://turtle/meshes/visual/Back_left1.STL" />
+          filename="package://turtle_on_land_demo/meshes/visual/Back_left1.STL" />
+      </geometry>
+      <material
+        name="">
+        <color
+          rgba="0 1 0 1" />
+      </material>
+    </visual>
+    <collision>
+      <origin
+        xyz="0 0 0"
+        rpy="0 0 0" />
+      <geometry>
+        <mesh
+          filename="package://turtle_on_land_demo/meshes/visual/Back_left1.STL" />
       </geometry>
     </collision>
@@ -504,7 +504,7 @@
       lower="-0.7854"
       upper="0.7854"
-      effort="2"
-      velocity="5" />
-    <dynamics damping="0.1" friction="0.1"/>
+      effort="10"
+      velocity="999" />
+    <dynamics damping="0.1" friction="5"/>
   </joint>
   <!--Link10;Back left flipper-->
@@ -531,19 +531,19 @@
       <geometry>
         <mesh
-          filename="package://turtle/meshes/visual/Back_left2.STL" />
-      </geometry>
-      <material
-        name="">
-        <color
-          rgba="0 1 0 1" />
-      </material>
-    </visual>
-    <collision>
-      <origin
-        xyz="0 0 0"
-        rpy="0 0 0" />
-      <geometry>
-        <mesh
-          filename="package://turtle/meshes/visual/Back_left2.STL" />
+          filename="package://turtle_on_land_demo/meshes/visual/Back_left2.STL" />
+      </geometry>
+      <material
+        name="">
+        <color
+          rgba="0 1 0 1" />
+      </material>
+    </visual>
+    <collision>
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