Commit message: Add files via upload
Updated URDF.xacro, xacro includes, damping and friction tags as well as updated velocity end effort tags.

File: Control/turtle/urdf/URDF1.urdf.xacro (robot description, xacro)
@@ -56,5 +56,5 @@
         <!--Filepath to STL visual Mesh file-->
       <geometry>
-        <mesh filename="package://meshes/visual/base_link.stl"/>
+        <mesh filename="package://turtle/meshes/visual/base_link.STL"/>
       </geometry>
       <material
@@ -64,5 +64,5 @@
           rgba="0 1 0 1" />
       </material>
-    </visual>s
+    </visual>
     <!--Collision parameter for Link-->
     <collision>
@@ -73,5 +73,5 @@
       <geometry>
         <mesh
-          filename="package://meshes/visual/base_link.stl" />
+          filename="package://turtle/meshes/visual/base_link.STL" />
       </geometry>
     </collision>
@@ -102,19 +102,19 @@
       <geometry>
         <mesh
-          filename="package://meshes/visual/Front_right1.stl" />
-      </geometry>
-      <material
-        name="">
-        <color
-          rgba="0 1 0 1" />
-      </material>
-    </visual>
-    <collision>
-      <origin
-        xyz="0 0 0"
-        rpy="0 0 0" />
-      <geometry>
-        <mesh
-          filename="package://meshes/visual/Front_right1.stl" />
+          filename="package://turtle/meshes/visual/Front_right1.STL" />
+      </geometry>
+      <material
+        name="">
+        <color
+          rgba="0 1 0 1" />
+      </material>
+    </visual>
+    <collision>
+      <origin
+        xyz="0 0 0"
+        rpy="0 0 0" />
+      <geometry>
+        <mesh
+          filename="package://turtle/meshes/visual/Front_right1.STL" />
       </geometry>
     </collision>
@@ -163,19 +163,19 @@
       <geometry>
         <mesh
-          filename="package://meshes/visual/Front_right2.stl" />
-      </geometry>
-      <material
-        name="">
-        <color
-          rgba="0 1 0 1" />
-      </material>
-    </visual>
-    <collision>
-      <origin
-        xyz="0 0 0"
-        rpy="0 0 0" />
-      <geometry>
-        <mesh
-          filename="package://meshes/visual/Front_right2.stl" />
+          filename="package://turtle/meshes/visual/Front_right2.STL" />
+      </geometry>
+      <material
+        name="">
+        <color
+          rgba="0 1 0 1" />
+      </material>
+    </visual>
+    <collision>
+      <origin
+        xyz="0 0 0"
+        rpy="0 0 0" />
+      <geometry>
+        <mesh
+          filename="package://turtle/meshes/visual/Front_right2.STL" />
       </geometry>
     </collision>
@@ -224,19 +224,19 @@
       <geometry>
         <mesh
-          filename="package://meshes/visual/Back_right1.stl" />
-      </geometry>
-      <material
-        name="">
-        <color
-          rgba="0 1 0 1" />
-      </material>
-    </visual>
-    <collision>
-      <origin
-        xyz="0 0 0"
-        rpy="0 0 0" />
-      <geometry>
-        <mesh
-          filename="package://meshes/visual/Back_right1.stl" />
+          filename="package://turtle/meshes/visual/Back_right1.STL" />
+      </geometry>
+      <material
+        name="">
+        <color
+          rgba="0 1 0 1" />
+      </material>
+    </visual>
+    <collision>
+      <origin
+        xyz="0 0 0"
+        rpy="0 0 0" />
+      <geometry>
+        <mesh
+          filename="package://turtle/meshes/visual/Back_right1.STL" />
       </geometry>
     </collision>
@@ -285,19 +285,19 @@
       <geometry>
         <mesh
-          filename="package://meshes/visual/Back_right2.stl" />
-      </geometry>
-      <material
-        name="">
-        <color
-          rgba="0 1 0 1" />
-      </material>
-    </visual>
-    <collision>
-      <origin
-        xyz="0 0 0"
-        rpy="0 0 0" />
-      <geometry>
-        <mesh
-          filename="package://meshes/visual/Back_right2.stl" />
+          filename="package://turtle/meshes/visual/Back_right2.STL" />
+      </geometry>
+      <material
+        name="">
+        <color
+          rgba="0 1 0 1" />
+      </material>
+    </visual>
+    <collision>
+      <origin
+        xyz="0 0 0"
+        rpy="0 0 0" />
+      <geometry>
+        <mesh
+          filename="package://turtle/meshes/visual/Back_right2.STL" />
       </geometry>
     </collision>
@@ -346,19 +346,19 @@
       <geometry>
         <mesh
-          filename="package://meshes/visual/Front_left1.stl" />
-      </geometry>
-      <material
-        name="">
-        <color
-          rgba="0 1 0 1" />
-      </material>
-    </visual>
-    <collision>
-      <origin
-        xyz="0 0 0"
-        rpy="0 0 0" />
-      <geometry>
-        <mesh
-          filename="package://meshes/visual/Front_left1.stl" />
+          filename="package://turtle/meshes/visual/Front_left1.STL" />
+      </geometry>
+      <material
+        name="">
+        <color
+          rgba="0 1 0 1" />
+      </material>
+    </visual>
+    <collision>
+      <origin
+        xyz="0 0 0"
+        rpy="0 0 0" />
+      <geometry>
+        <mesh
+          filename="package://turtle/meshes/visual/Front_left1.STL" />
       </geometry>
     </collision>
@@ -378,6 +378,6 @@
       xyz="0 0 -1" />
     <limit
-      lower="-0.7854"
-      upper="0.7854"
+      lower="-0.6854"
+      upper="0.6854"
       effort="2"
       velocity="5" />
@@ -407,19 +407,19 @@
       <geometry>
         <mesh
-          filename="package://meshes/visual/Front_left2.stl" />
-      </geometry>
-      <material
-        name="">
-        <color
-          rgba="0 1 0 1" />
-      </material>
-    </visual>
-    <collision>
-      <origin
-        xyz="0 0 0"
-        rpy="0 0 0" />
-      <geometry>
-        <mesh
-          filename="package://meshes/visual/Front_left2.stl" />
+          filename="package://turtle/meshes/visual/Front_left2.STL" />
+      </geometry>
+      <material
+        name="">
+        <color
+          rgba="0 1 0 1" />
+      </material>
+    </visual>
+    <collision>
+      <origin
+        xyz="0 0 0"
+        rpy="0 0 0" />
+      <geometry>
+        <mesh
+          filename="package://turtle/meshes/visual/Front_left2.STL" />
       </geometry>
     </collision>
@@ -468,19 +468,19 @@
       <geometry>
         <mesh
-          filename="package://meshes/visual/Back_left1.stl" />
-      </geometry>
-      <material
-        name="">
-        <color
-          rgba="0 1 0 1" />
-      </material>
-    </visual>
-    <collision>
-      <origin
-        xyz="0 0 0"
-        rpy="0 0 0" />
-      <geometry>
-        <mesh
-          filename="package://meshes/visual/Back_left1.stl" />
+          filename="package://turtle/meshes/visual/Back_left1.STL" />
+      </geometry>
+      <material
+        name="">
+        <color
+          rgba="0 1 0 1" />
+      </material>
+    </visual>
+    <collision>
+      <origin
+        xyz="0 0 0"
+        rpy="0 0 0" />
+      <geometry>
+        <mesh
+          filename="package://turtle/meshes/visual/Back_left1.STL" />
       </geometry>
     </collision>
@@ -529,19 +529,19 @@
       <geometry>
         <mesh
-          filename="package://meshes/visual/Back_left2.stl" />
-      </geometry>
-      <material
-        name="">
-        <color
-          rgba="0 1 0 1" />
-      </material>
-    </visual>
-    <collision>
-      <origin
-        xyz="0 0 0"
-        rpy="0 0 0" />
-      <geometry>
-        <mesh
-          filename="package://meshes/visual/Back_left2.stl" />
+          filename="package://turtle/meshes/visual/Back_left2.STL" />
+      </geometry>
+      <material
+        name="">
+        <color
+          rgba="0 1 0 1" />
+      </material>
+    </visual>
+    <collision>
+      <origin
+        xyz="0 0 0"
+        rpy="0 0 0" />
+      <geometry>
+        <mesh
+          filename="package://turtle/meshes/visual/Back_left2.STL" />
       </geometry>
     </collision>
@@ -567,3 +567,36 @@
     <dynamics damping="0.1" friction="0.1"/>
   </joint>
+  <link
+    name="Sensor_link">
+    <inertial>
+      <origin
+        xyz="-2.25214372452731E-05 0.103607028948444 -0.00174327710854269"
+        rpy="0 0 0" />
+      <mass
+        value="0.656382274118652" />
+      <inertia
+        ixx="0.00398589796619268"
+        ixy="6.81523498247126E-07"
+        ixz="7.5942173311683E-08"
+        iyy="0.00261594481266056"
+        iyz="4.49451871288875E-05"
+        izz="0.00597901119561345" />
+    </inertial>
+  </link>
+  <joint
+    name="sensor"
+    type="fixed">
+    <origin
+      xyz="0.0975 0 0.005"
+      rpy="0 0 0" />
+    <parent
+      link="base_link" />
+    <child
+      link="Sensor_link" />
+    <axis
+      xyz="0 0 0" />
+  </joint>
+  <plugin name="lidar" filename="libgazebo_ros_ray_sensor.so">
+    <output_type>sensor_msgs/LaserScan</output_type>
+  </plugin>
 </robot>

Commit message: Add files via upload

File: Control/turtle/urdf/URDF1.urdf.xacro (robot description, xacro)
@@ -601,3 +601,35 @@
       xyz="0 0 0" />
   </joint>
+  <!--Camera Link-->
+  <link
+    name="Camera_link">
+    <inertial>
+      <origin
+        xyz="-2.25214372452731E-05 0.103607028948444 -0.00174327710854269"
+        rpy="0 0 0" />
+      <mass
+        value="0.656382274118652" />
+      <inertia
+        ixx="0.00398589796619268"
+        ixy="6.81523498247126E-07"
+        ixz="7.5942173311683E-08"
+        iyy="0.00261594481266056"
+        iyz="4.49451871288875E-05"
+        izz="0.00597901119561345" />
+    </inertial>
+  </link>
+  <!--Camera_Joint-->
+   <joint
+    name="camera"
+    type="fixed">
+    <origin
+      xyz="0.0975 0 0.005"
+      rpy="0 0 0" />
+    <parent
+      link="base_link" />
+    <child
+      link="Camera_link" />
+    <axis
+      xyz="0 0 0" />
+  </joint>
 </robot>

Commit message: Updated URDF and Publisher

File: Control/turtle/urdf/URDF1.urdf.xacro (robot description, xacro)
@@ -2,14 +2,8 @@
 <!-- Turtle on land URDF file-->
 <robot name="URDF1" xmlns:xacro="http://www.ros.org/wiki/xacro">
-<<<<<<< HEAD
   <!-- Import turtle ros2_control description -->
-  <xacro:include filename="$(find turtle_on_land_demo)/src/ros2_control.xacro" />
+  <xacro:include filename="$(find turtle)/src/ros2_control.xacro" />
   <!-- Import turtle gazebo sensor descriptions -->
-=======
-  <!-- Import turtlebot ros2_control description -->
-  <xacro:include filename="$(find turtle_on_land_demo)/src/ros2_control.xacro" />
-  <!-- Import turtle gazebo lidar description -->
->>>>>>> 1e033910d575f7fe92138ab8b5531f3dbd53b3d7
-  <xacro:include filename="$(find turtle_on_land_demo)/gazebo/turtle.gazebo.xacro" />
+  <xacro:include filename="$(find turtle)/gazebo/turtle.gazebo.xacro" />
   <!--Link1; Turtle Shell bottom-->
   <link name="base_footprint">
@@ -146,9 +140,5 @@
       effort="20"
       velocity="999" />
-<<<<<<< HEAD
-    <dynamics damping="0.1" friction="5"/>
-=======
-    <dynamics damping="0.1" friction="0.1"/>
->>>>>>> 1e033910d575f7fe92138ab8b5531f3dbd53b3d7
+    <dynamics damping="0.1" friction="5"/>
   </joint>
   <!--Link4; Froint right flipper-->
@@ -211,9 +201,5 @@
       effort="20"
       velocity="999" />
-<<<<<<< HEAD
-    <dynamics damping="0.1" friction="5"/>
-=======
-    <dynamics damping="0.1" friction="0.1"/>
->>>>>>> 1e033910d575f7fe92138ab8b5531f3dbd53b3d7
+    <dynamics damping="0.1" friction="5"/>
   </joint>
   <!--Link5; Back right shoulder-->
@@ -276,9 +262,5 @@
       effort="10"
       velocity="999" />
-<<<<<<< HEAD
-    <dynamics damping="0.1" friction="5"/>
-=======
-    <dynamics damping="0.1" friction="0.1"/>
->>>>>>> 1e033910d575f7fe92138ab8b5531f3dbd53b3d7
+    <dynamics damping="0.1" friction="5"/>
   </joint>
   <!--Link6; Back right flipper-->
@@ -341,9 +323,5 @@
       effort="10"
       velocity="999" />
-<<<<<<< HEAD
-    <dynamics damping="0.1" friction="5"/>
-=======
-    <dynamics damping="0.1" friction="0.1"/>
->>>>>>> 1e033910d575f7fe92138ab8b5531f3dbd53b3d7
+    <dynamics damping="0.1" friction="5"/>
   </joint>
   <!--Link7; Front left shoulder-->
@@ -406,9 +384,5 @@
       effort="20"
       velocity="999" />
-<<<<<<< HEAD
-    <dynamics damping="0.1" friction="5"/>
-=======
-    <dynamics damping="0.1" friction="0.1"/>
->>>>>>> 1e033910d575f7fe92138ab8b5531f3dbd53b3d7
+    <dynamics damping="0.1" friction="5"/>
   </joint>
   <!--Link8; Front left flipper-->
@@ -471,9 +445,5 @@
       effort="20"
       velocity="999" />
-<<<<<<< HEAD
-    <dynamics damping="0.1" friction="5"/>
-=======
-    <dynamics damping="0.1" friction="0.1"/>
->>>>>>> 1e033910d575f7fe92138ab8b5531f3dbd53b3d7
+    <dynamics damping="0.1" friction="5"/>
   </joint>
   <!--Link9; Back left shoulder-->
@@ -536,9 +506,5 @@
       effort="10"
       velocity="999" />
-<<<<<<< HEAD
-    <dynamics damping="0.1" friction="5"/>
-=======
-    <dynamics damping="0.1" friction="0.1"/>
->>>>>>> 1e033910d575f7fe92138ab8b5531f3dbd53b3d7
+    <dynamics damping="0.1" friction="5"/>
   </joint>
   <!--Link10;Back left flipper-->
@@ -601,9 +567,5 @@
       effort="10"
       velocity="999" />
-<<<<<<< HEAD
-    <dynamics damping="0.1" friction="5"/>
-=======
-    <dynamics damping="0.1" friction="0.1"/>
->>>>>>> 1e033910d575f7fe92138ab8b5531f3dbd53b3d7
+    <dynamics damping="0.1" friction="5"/>
   </joint>
   <link
